Commit message: clean-up urdf

File: assets/urdf/ur5_robotiq_85.urdf (robot description, URDF)
Before this commit: robot ur5_robotiq_85, 20 links, 19 joints
Joints:
- joint ee_fixed_joint: origin xyz=0.0 0.0823 0.0 rpy=0.0 0.0 1.57079632679 -> xyz=0.0 0.0823 0.0 rpy=0 0 1.57079632679
- joint elbow_joint: origin xyz=0.0 -0.1197 0.425 rpy=0.0 0.0 0.0 -> xyz=0.0 -0.1197 0.425 rpy=0 0 0
- joint shoulder_lift_joint: origin xyz=0.0 0.13585 0.0 rpy=0.0 1.57079632679 0.0 -> xyz=0.0 0.13585 0.0 rpy=0 1.57079632679 0
- joint shoulder_pan_joint: origin xyz=0.0 0.0 0.089159 rpy=0.0 0.0 0.0 -> xyz=0.0 0.0 0.089159 rpy=0 0 0
- joint world_arm_joint: origin xyz=0 0 0 rpy=0.0 0.0 0 -> xyz=0 0 0 rpy=0 0 0
- joint wrist_1_joint: origin xyz=0.0 0.0 0.39225 rpy=0.0 1.57079632679 0.0 -> xyz=0.0 0.0 0.39225 rpy=0 1.57079632679 0
- joint wrist_2_joint: origin xyz=0.0 0.093 0.0 rpy=0.0 0.0 0.0 -> xyz=0.0 0.093 0.0 rpy=0 0 0
- joint wrist_3_joint: origin xyz=0.0 0.0 0.09465 rpy=0.0 0.0 0.0 -> xyz=0.0 0.0 0.09465 rpy=0 0 0

Commit message: add tcp_link to the robot

File: assets/urdf/ur5_robotiq_85.urdf (robot description, URDF)
Before this commit: robot ur5_robotiq_85, 20 links, 19 joints
Links:
- added link tcp_link, mass 0.0001; collision box size=0.001 0.001 0.001; visual box size=0.001 0.001 0.001
Joints:
- added joint tcp_joint: type fixed, parent ee_link, child tcp_link, origin xyz=0.145 0.0 0.0 rpy=0 0 0
