Commit message: clean up the code

File: assets/urdf/panda.urdf (robot description, URDF)
Before this commit: robot panda, 13 links, 12 joints
Links:
- added link tcp_link; visual box size=0.001 0.001 0.001
Joints:
- added joint tcp_joint: type fixed, parent panda_grasptarget, child tcp_link, origin xyz=0.0 0.0 0.0 rpy=0 0 0

File: assets/urdf/ur5_robotiq_85.urdf (robot description, URDF)
Before this commit: robot ur5_robotiq_85, 21 links, 20 joints
Links:
- link tcp_link: mass 0.0001 -> None; geometry visual box size=0.001 0.001 0.001

Commit message: transform the frame of tcp_link in the urdf

File: assets/urdf/panda.urdf (robot description, URDF)
Before this commit: robot panda, 14 links, 13 joints
Joints:
- joint tcp_joint: origin xyz=0.0 0.0 0.0 rpy=0 0 0 -> xyz=0.0 0.0 0.0 rpy=3.1415927 0 0

Commit message: np.array

File: assets/urdf/panda.urdf (robot description, URDF)
Before this commit: robot panda, 14 links, 13 joints
Links:
- link tcp_link: mass None -> 0.0
